File: pcb/base/base.sch (KiCad schematic (older format))
At the start: 21 parts, among them J1 Conn_01x03_Male, J2 Conn_01x03_Male, J3 Conn_01x02_Male, J4 Conn_01x03_Male, U1 STM32G431KBT6, U2 AP2210-33, U3 tile

Commit message: cleaning/upgrades got collection of little modes over sime time, added dxf"
Parts:
- removed C1: 10uf, Capacitors_SMD:C_0603_HandSoldering, symbol Device:C_Small
- removed C2, C3: 4.7uf, Capacitors_SMD:C_0603_HandSoldering, symbol Device:C_Small
- removed J1, J2: Conn_01x03_Male, Connectors_JST:JST_PH_B3B-PH-K_03x2.00mm_Straight, symbol Connector:Conn_01x03_Male
- removed U2: AP2210-33, TO_SOT_Packages_SMD:SOT-23-5_HandSoldering, symbol Regulator_Linear:AP1117-33
- C4, C6, C9: footprint Capacitors_SMD:C_0603_HandSoldering -> Capacitor_SMD:C_0603_1608Metric_Pad1.05x0.95mm_HandSolder
- D1, D2: footprint LEDs:LED_0603_HandSoldering -> LED_SMD:LED_0603_1608Metric_Pad1.05x0.95mm_HandSolder
- Hole1, Hole2: footprint Mounting_Holes:MountingHole_2.2mm_M2 -> MountingHole:MountingHole_2.2mm_M2
- J3: footprint Pin_Headers:Pin_Header_Straight_1x02_Pitch1.27mm -> Connector_PinHeader_1.27mm:PinHeader_1x02_P1.27mm_Vertical
- J4: footprint Pin_Headers:Pin_Header_Straight_1x03_Pitch1.27mm -> Connector_PinHeader_1.27mm:PinHeader_1x03_P1.27mm_Vertical
- R1, R3, R4, R6: footprint Resistors_SMD:R_0603_HandSoldering -> Resistor_SMD:R_0603_1608Metric_Pad1.05x0.95mm_HandSolder
- U1: footprint Housings_QFP:LQFP-32_7x7mm_Pitch0.8mm -> Package_QFP:LQFP-32_7x7mm_P0.8mm
Connections:
- net +3V3: no longer U3.2 (3V3), U3.3 (3V3), U3.4 (3V3)
- net ADC0: now also U3.16 (TX); no longer U3.32 (ADC0)
- net ADC1: now also U3.15 (RX); no longer U3.31 (ADC1)
- net BUS: now also U3.11 (PB4)
- net CRX: now also U3.6 (GND); no longer U3.14 (CRX)
- net CTX: now also U3.5 (GND); no longer U3.13 (CTX)
- net GND: now also U3.10 (SCL), U3.2 (3V3); no longer U3.17 (GND), U3.18 (GND), U3.19 (GND), U3.20 (GND), U3.5 (GND), U3.6 (GND), U3.7 (GND), U3.8 (GND)
- net I2C_CLK: now also U3.4 (3V3); no longer U3.10 (SCL)
- net I2C_SDA: now also U3.3 (3V3); no longer U3.9 (SDA)
- net PA3: no longer U3.30 (PA3)
- net PA4: no longer U3.29 (PA4)
- net PB0: no longer U3.25 (PB0)
- net PB3: no longer U3.12 (PB3)
- net PB4: no longer U3.11 (PB4)
- net SPI_CLK: now also U3.14 (CRX); no longer U3.28 (SCLK)
- net SPI_MISO: now also U3.13 (CTX); no longer U3.27 (MISO)
- net SPI_MOSI: now also U3.12 (PB3); no longer U3.26 (MOSI)
- net USART1_RX: now also U3.7 (GND); no longer U3.15 (RX)
- net USART1_TX: now also U3.8 (GND); no longer U3.16 (TX)
- net VCC: now also U3.9 (SDA); no longer U3.21 (VCC), U3.22 (VCC), U3.23 (VCC), U3.24 (VCC)
